File: zx-interface-2-rom.kicad_pcb (KiCad board)
At the start: 2 copper layers, 39.4 x 50.1 mm, 9 parts, among them J1 cartridge_IF2, SW1 ROM select, U1 W27C512, U2 74LS32

Commit message: version 1.2
Parts:
- removed G200: LOGO, ZXINFO_FOOTPRINT:ZXInfo_kicad_logo_copper_16.5x5
- moved J1 0.25 mm to (111.1, 92.1)
- moved SW1 0.22 mm to (116.8, 56.3)
Connections:
- R1 pad 1: +5V -> GND
- R2 pad 1: +5V -> GND
- SW1 pad 1: GND -> Net-(U1-A15)
- SW1 pad 2: GND -> Net-(U1-A14)
- SW1 pad 3: Net-(U1-A14) -> +5V
- SW1 pad 4: Net-(U1-A15) -> +5V
Routing:
- net D3: track 96.2 -> 50.2 mm, vias 0 -> 1
- net D4: track 49.5 -> 77.3 mm
- net Net-(J1-A15): track 80.5 -> 54.0 mm
- net D6: track 62.8 -> 37.6 mm, vias 0 -> 1
- net +5V: track 117.6 -> 98.4 mm, vias 0 -> 1
- net D7: track 43.1 -> 34.7 mm
- net Net-(U1-A14): track 38.6 -> 45.3 mm
- net A4: track 16.8 -> 22.2 mm, vias 3 -> 0
- net A13: track 46.2 -> 41.2 mm
- net D5: track 46.3 -> 41.3 mm
- net D2: track 48.7 -> 44.1 mm
- net D0: track 37.2 -> 32.8 mm
- net D1: track 42.9 -> 38.5 mm
- net A8: track 40.8 -> 36.9 mm
- net A12: track 41.2 -> 44.9 mm, vias 0 -> 1
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Other:
- board text added: "JLCJLCJLCJLC"
- board text added: "zx-interface-2-rom v1.2 - by ZXINFO"
