File: zx-interface-2-rom.kicad_sch (KiCad schematic)
At the start: 8 parts, among them J1 cartridge_IF2, SW1 SW_DIP_x02, U1 W27C512, U2 74LS32

Commit message: Updated SYMBOL & FOOTPRINT library
Parts:
- J1: footprint ZXINFO_LIB:ZX_I2_ROM_EDGE_CONNECTOR_V2 -> ZXINFO_FOOTPRINT:CART_IF2_EDGE; symbol ZXINFO_LIB:cartridge_IF2 -> ZXINFO_SYMBOL:cartridge_IF2
- U1: symbol ZXINFO_LIB:W27C512 -> ZXINFO_SYMBOL:W27C512
Changed lines of the file:
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@@
 		)
 		(instances
-			(project "ZX-Interface-2-ZXINFO"
+			(project "zx-interface-2-rom"
 				(path "/f29e48fc-2e79-4af0-a809-41de68718d80"
 					(reference "R1")
@@
 	)
 	(symbol
-		(lib_id "ZXINFO_LIB:cartridge_IF2")
+		(lib_id "ZXINFO_SYMBOL:cartridge_IF2")
 		(at 50.8 106.68 0)
 		(unit 1)
@@
 			)
 		)
-		(property "Footprint" "ZXINFO_LIB:ZX_I2_ROM_EDGE_CONNECTOR_V2"
+		(property "Footprint" "ZXINFO_FOOTPRINT:CART_IF2_EDGE"
 			(at 80.01 106.68 0)
 			(effects
@@
 		)
 		(instances
-			(project "ZX-Interface-2-ZXINFO"
+			(project "zx-interface-2-rom"
 				(path "/f29e48fc-2e79-4af0-a809-41de68718d80"
 					(reference "J1")
@@
 		)
 		(instances
-			(project "ZX-Interface-2-ZXINFO"
+			(project "zx-interface-2-rom"
 				(path "/f29e48fc-2e79-4af0-a809-41de68718d80"
 					(reference "#PWR010")
@@
 		)
 		(instances
-			(project "ZX-Interface-2-ZXINFO"
+			(project "zx-interface-2-rom"
 				(path "/f29e48fc-2e79-4af0-a809-41de68718d80"
 					(reference "C2")
@@
 		)
 		(instances
-			(project "ZX-Interface-2-ZXINFO"
+			(project "zx-interface-2-rom"
 				(path "/f29e48fc-2e79-4af0-a809-41de68718d80"
 					(reference "R2")
@@
 		)
 		(instances
-			(project "ZX-Interface-2-ZXINFO"
+			(project "zx-interface-2-rom"
 				(path "/f29e48fc-2e79-4af0-a809-41de68718d80"
 					(reference "U2")
@@
 		)
 		(instances
-			(project "ZX-Interface-2-ZXINFO"
+			(project "zx-interface-2-rom"
 				(path "/f29e48fc-2e79-4af0-a809-41de68718d80"
 					(reference "SW1")
@@
 		)
 		(instances
-			(project "ZX-Interface-2-ZXINFO"
+			(project "zx-interface-2-rom"
 				(path "/f29e48fc-2e79-4af0-a809-41de68718d80"
 					(reference "U2")
@@
 		)
 		(instances
-			(project "ZX-Interface-2-ZXINFO"
+			(project "zx-interface-2-rom"
 				(path "/f29e48fc-2e79-4af0-a809-41de68718d80"
 					(reference "#PWR06")
@@
 		)
 		(instances
-			(project "ZX-Interface-2-ZXINFO"
+			(project "zx-interface-2-rom"
 				(path "/f29e48fc-2e79-4af0-a809-41de68718d80"
 					(reference "#PWR01")
@@
 		)
 		(instances
-			(project "ZX-Interface-2-ZXINFO"
+			(project "zx-interface-2-rom"
 				(path "/f29e48fc-2e79-4af0-a809-41de68718d80"
 					(reference "#PWR09")
@@
 		)
 		(instances
-			(project "ZX-Interface-2-ZXINFO"
+			(project "zx-interface-2-rom"
 				(path "/f29e48fc-2e79-4af0-a809-41de68718d80"
 					(reference "#PWR07")
@@
 		)
 		(instances
-			(project "ZX-Interface-2-ZXINFO"
+			(project "zx-interface-2-rom"
 				(path "/f29e48fc-2e79-4af0-a809-41de68718d80"
 					(reference "U2")
@@
 		)
 		(instances
-			(project "ZX-Interface-2-ZXINFO"
+			(project "zx-interface-2-rom"
 				(path "/f29e48fc-2e79-4af0-a809-41de68718d80"
 					(reference "#FLG02")
@@
 	)
 	(symbol
-		(lib_id "ZXINFO_LIB:W27C512")
+		(lib_id "ZXINFO_SYMBOL:W27C512")
 		(at 129.54 74.93 0)
 		(unit 1)
@@
 		)
 		(instances
-			(project "ZX-Interface-2-ZXINFO"
+			(project "zx-interface-2-rom"
 				(path "/f29e48fc-2e79-4af0-a809-41de68718d80"
 					(reference "U1")
@@
 		)
 		(instances
-			(project "ZX-Interface-2-ZXINFO"
+			(project "zx-interface-2-rom"
 				(path "/f29e48fc-2e79-4af0-a809-41de68718d80"
 					(reference "#PWR04")
@@
 		)
 		(instances
-			(project "ZX-Interface-2-ZXINFO"
+			(project "zx-interface-2-rom"
 				(path "/f29e48fc-2e79-4af0-a809-41de68718d80"
 					(reference "U2")
@@
 		)
 		(instances
-			(project "ZX-Interface-2-ZXINFO"
+			(project "zx-interface-2-rom"
 				(path "/f29e48fc-2e79-4af0-a809-41de68718d80"
 					(reference "#PWR02")
@@
 		)
 		(instances
-			(project "ZX-Interface-2-ZXINFO"
+			(project "zx-interface-2-rom"
 				(path "/f29e48fc-2e79-4af0-a809-41de68718d80"
 					(reference "U2")
@@
 		)
 		(instances
-			(project "ZX-Interface-2-ZXINFO"
+			(project "zx-interface-2-rom"
 				(path "/f29e48fc-2e79-4af0-a809-41de68718d80"
 					(reference "#FLG01")
@@
 		)
 		(instances
-			(project "ZX-Interface-2-ZXINFO"
+			(project "zx-interface-2-rom"
 				(path "/f29e48fc-2e79-4af0-a809-41de68718d80"
 					(reference "C1")
@@
 		)
 		(instances
-			(project "ZX-Interface-2-ZXINFO"
+			(project "zx-interface-2-rom"
 				(path "/f29e48fc-2e79-4af0-a809-41de68718d80"
 					(reference "#PWR03")
@@
 		)
 		(instances
-			(project "ZX-Interface-2-ZXINFO"
+			(project "zx-interface-2-rom"
 				(path "/f29e48fc-2e79-4af0-a809-41de68718d80"
 					(reference "#PWR05")
@@
 		)
 		(instances
-			(project "ZX-Interface-2-ZXINFO"
+			(project "zx-interface-2-rom"
 				(path "/f29e48fc-2e79-4af0-a809-41de68718d80"
 					(reference "#PWR08")

Commit message: version 2 - added solder mask to pad
Parts:
- R1: value 4K7 -> 10K
- R2: value 4K7 -> 10K; footprint R_Axial_DIN0207_L6.3mm_D2.5mm_P10.16mm_Horizontal -> Resistor_THT:R_Axial_DIN0207_L6.3mm_D2.5mm_P10.16mm_Horizontal
- SW1: value SW_DIP_x02 -> ROM select
Connections:
- net at R1.2, U1.1 (A15): now also SW1.4; no longer SW1.3
- net at R2.2, U1.27 (A14): now also SW1.3; no longer SW1.4
Changed lines of the file:
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@@
+	)
+	(junction
+		(at 96.52 44.45)
+		(diameter 0)
+		(color 0 0 0 0)
+	)
+	(junction
+		(at 78.74 156.21)
+		(diameter 0)
+		(color 0 0 0 0)
+	)
+	(junction
+		(at 67.31 62.23)
+		(diameter 0)
+		(color 0 0 0 0)
+	)
+	(junction
+		(at 129.54 38.1)
+		(diameter 0)
+		(color 0 0 0 0)
+	)
+	(junction
+		(at 73.66 88.9)
+		(diameter 0)
+		(color 0 0 0 0)
+	)
+	(junction
+		(at 36.83 139.7)
+		(diameter 0)
+		(color 0 0 0 0)
 	)
 	(junction
@@
 	)
 	(junction
-		(at 96.52 44.45)
-		(diameter 0)
-		(color 0 0 0 0)
-	)
-	(junction
-		(at 78.74 156.21)
-		(diameter 0)
-		(color 0 0 0 0)
-	)
-	(junction
-		(at 68.58 62.23)
-		(diameter 0)
-		(color 0 0 0 0)
-	)
-	(junction
-		(at 129.54 38.1)
-		(diameter 0)
-		(color 0 0 0 0)
-	)
-	(junction
-		(at 73.66 88.9)
-		(diameter 0)
-		(color 0 0 0 0)
-	)
-	(junction
-		(at 36.83 139.7)
-		(diameter 0)
-		(color 0 0 0 0)
-	)
-	(junction
 		(at 36.83 152.4)
 		(diameter 0)
@@
 	(wire
 		(pts
+			(xy 90.17 62.23) (xy 96.52 62.23)
+		)
+		(stroke
+			(width 0)
+			(type default)
+		)
+	)
+	(wire
+		(pts
 			(xy 109.22 59.69) (xy 109.22 81.28)
 		)
@@
 	(wire
 		(pts
-			(xy 68.58 59.69) (xy 68.58 62.23)
+			(xy 67.31 59.69) (xy 67.31 62.23)
 		)
 		(stroke
@@
 	(wire
 		(pts
-			(xy 60.96 62.23) (xy 68.58 62.23)
+			(xy 59.69 62.23) (xy 67.31 62.23)
 		)
 		(stroke
@@
 	(wire
 		(pts
-			(xy 68.58 62.23) (xy 74.93 62.23)
-		)
-		(stroke
-			(width 0)
-			(type default)
-		)
-	)
-	(wire
-		(pts
 			(xy 73.66 88.9) (xy 78.74 88.9)
 		)
@@
 	(wire
 		(pts
-			(xy 68.58 66.04) (xy 68.58 62.23)
+			(xy 67.31 66.04) (xy 67.31 62.23)
 		)
 		(stroke
@@
 	(wire
 		(pts
-			(xy 96.52 62.23) (xy 90.17 62.23)
-		)
-		(stroke
-			(width 0)
-			(type default)
-		)
-	)
-	(wire
-		(pts
 			(xy 63.5 106.68) (xy 73.66 106.68)
 		)
@@
 	(wire
 		(pts
+			(xy 67.31 62.23) (xy 74.93 62.23)
+		)
+		(stroke
+			(width 0)
+			(type default)
+		)
+	)
+	(wire
+		(pts
 			(xy 88.9 99.06) (xy 88.9 101.6)
 		)
@@
 	(wire
 		(pts
-			(xy 74.93 59.69) (xy 68.58 59.69)
+			(xy 74.93 59.69) (xy 67.31 59.69)
 		)
 		(stroke
@@
 			)
 		)
-		(property "Value" "4K7"
+		(property "Value" "10K"
 			(at 99.06 53.3399 0)
 			(effects
@@
 			)
 		)
-		(property "Value" "4K7"
+		(property "Value" "10K"
 			(at 106.68 53.3399 0)
 			(effects
@@
 			)
 		)
-		(property "Footprint" "R_Axial_DIN0207_L6.3mm_D2.5mm_P10.16mm_Horizontal"
+		(property "Footprint" "Resistor_THT:R_Axial_DIN0207_L6.3mm_D2.5mm_P10.16mm_Horizontal"
 			(at 102.362 52.07 90)
 			(effects
@@
 	(symbol
 		(lib_id "Switch:SW_DIP_x02")
-		(at 82.55 62.23 0)
+		(at 82.55 59.69 0)
+		(mirror x)
 		(unit 1)
 		(exclude_from_sim no)
@@
 		(dnp no)
 		(property "Reference" "SW1"
-			(at 82.55 52.07 0)
-			(effects
-				(font
-					(size 1.27 1.27)
-				)
-			)
-		)
-		(property "Value" "SW_DIP_x02"
-			(at 82.55 54.61 0)
+			(at 82.55 69.85 0)
+			(effects
+				(font
+					(size 1.27 1.27)
+				)
+			)
+		)
+		(property "Value" "ROM select"
+			(at 82.55 67.31 0)
 			(effects
 				(font
@@
 		)
 		(property "Footprint" "Button_Switch_THT:SW_DIP_SPSTx02_Slide_6.7x6.64mm_W7.62mm_P2.54mm_LowProfile"
-			(at 82.55 62.23 0)
+			(at 82.55 59.69 0)
 			(effects
 				(font
@@
 		)
 		(property "Datasheet" "~"
-			(at 82.55 62.23 0)
+			(at 82.55 59.69 0)
 			(effects
 				(font
@@
 		)
 		(property "Description" "2x DIP Switch, Single Pole Single Throw (SPST) switch, small symbol"
-			(at 82.55 62.23 0)
+			(at 82.55 59.69 0)
 			(effects
 				(font
@@
 	(symbol
 		(lib_id "power:GND")
-		(at 68.58 66.04 0)
+		(at 67.31 66.04 0)
 		(unit 1)
 		(exclude_from_sim no)
@@
 		(fields_autoplaced yes)
 		(property "Reference" "#PWR02"
-			(at 68.58 72.39 0)
+			(at 67.31 72.39 0)
 			(effects
 				(font
@@
 		)
 		(property "Value" "GND"
-			(at 68.58 71.12 0)
+			(at 67.31 71.12 0)
 			(effects
 				(font
@@
 		)
 		(property "Footprint" ""
-			(at 68.58 66.04 0)
+			(at 67.31 66.04 0)
 			(effects
 				(font
@@
 		)
 		(property "Datasheet" ""
-			(at 68.58 66.04 0)
+			(at 67.31 66.04 0)
 			(effects
 				(font
@@
 		)
 		(property "Description" "Power symbol creates a global label with name \"GND\" , ground"
-			(at 68.58 66.04 0)
+			(at 67.31 66.04 0)
 			(effects
 				(font
@@
 	(symbol
 		(lib_id "power:PWR_FLAG")
-		(at 60.96 62.23 0)
+		(at 59.69 62.23 0)
 		(unit 1)
 		(exclude_from_sim no)
@@
 		(fields_autoplaced yes)
 		(property "Reference" "#FLG01"
-			(at 60.96 60.325 0)
+			(at 59.69 60.325 0)
 			(effects
 				(font
@@
 		)
 		(property "Value" "PWR_FLAG"
-			(at 60.96 57.15 0)
+			(at 59.69 57.15 0)
 			(effects
 				(font
@@
 		)
 		(property "Footprint" ""
-			(at 60.96 62.23 0)
+			(at 59.69 62.23 0)
 			(effects
 				(font
@@
 		)
 		(property "Datasheet" "~"
-			(at 60.96 62.23 0)
+			(at 59.69 62.23 0)
 			(effects
 				(font
@@
 		)
 		(property "Description" "Special symbol for telling ERC where power comes from"
-			(at 60.96 62.23 0)
-			(effects
-				(font
+			(at 59.69 62.23 0)
+			(effects
+				(font

Commit message: version 1.2
Connections:
- net +5V: now also SW1.3, SW1.4; no longer R1.1, R2.1
- net GND: now also R1.1, R2.1; no longer SW1.1, SW1.2
- net at R1.2, U1.1 (A15): now also SW1.1; no longer SW1.4
- net at R2.2, U1.27 (A14): now also SW1.2; no longer SW1.3
Other:
- moved on the sheet: SW1
